File: shieldV1/shieldV1/shieldV1.sch (KiCad schematic (older format))
At the start: 7 parts, among them J1 Conn_02x19_Odd_Even, J2 Conn_02x19_Odd_Even, J3 Conn_01x04_Female, J4 Conn_01x04_Female, J5 Conn_01x03_Female

Commit message: Add hall sensor PCB
Parts:
- added C1, C2: C, Capacitor_SMD:C_0603_1608Metric, symbol Device:C
- added J10: Conn_01x07_Female, Connector_JST:JST_GH_SM07B-GHS-TB_1x07-1MP_P1.25mm_Horizontal, symbol Connector:Conn_01x07_Female
- added J6, J7: Conn_01x03_Female, Connector_JST:JST_GH_SM03B-GHS-TB_1x03-1MP_P1.25mm_Horizontal, symbol Connector:Conn_01x03_Female
- added J8, J9: Conn_01x02_Female, Connector_JST:JST_GH_SM02B-GHS-TB_1x02-1MP_P1.25mm_Horizontal, symbol Connector:Conn_01x02_Female
- added JP2, JP3, JP4: SolderJumper_3_Open, Jumper:SolderJumper-3_P1.3mm_Open_RoundedPad1.0x1.5mm, symbol Jumper:SolderJumper_3_Open
- added R2, R3, R4, R5: 10K, Resistor_SMD:R_0603_1608Metric, symbol Device:R
Connections:
- net labels added: +5V, PA1_ADC1_1, PA_0_ADC1_0, PA_12_UART6_RX, PB1, PB2, PB3_SPI1_SCLK, PB4_SPI1_MISO, PB5_SPI1_MOSI, PB8_I2C1_SCL, PB9_I2C1_SDA, PC14, PC15
- net labels removed: E5V, PA_11_UART6_RX
- wire segments 25 -> 60
Other:
- note added: "I2C/SPI LCD"
- note added: "POT0\n"
- note added: "POT1\n"
- note added: "SWITCH0\n"
- note added: "SWITCH1\n"
- note added: "UART VESC0"
- note removed: "UART VESC2"
- moved on the sheet: J1, J3, J4, J5, JP1, R1
