File: BCU/mcu.kicad_sch (KiCad schematic)
At the start: 12 parts

Commit message: Make rough component placement for evaluating missing 3D
Parts:
- removed IC?: STM32G474RET6, QFP50P1200X1200X160-64N, symbol coilchain-mcu:STM32G474RET6
- added IC3: STM32G474RET6, Package_QFP:LQFP-64_10x10mm_P0.5mm, symbol coilchain-mcu:STM32G474RET6
- Y1: renamed from Y?; footprint (none) -> Crystal:Crystal_SMD_2520-4Pin_2.5x2.0mm
- gave numbers to parts that had none: 10
Connections:
- net +3V3: now also IC3.1 (VBAT), IC3.16 (VDD_1), IC3.28 (VREF+), IC3.29 (VDDA), IC3.32 (VDD_2), IC3.48 (VDD_3), IC3.64 (VDD_4)
- net ADC_BRAKE: now also IC3.13 (PA1)
- net ADC_THROT: now also IC3.14 (PA2)
- net ADC_TORQUE: now also IC3.17 (PA3)
- net BTN_DOWN: now also IC3.9 (PC1)
- net BTN_LEFT: now also IC3.10 (PC2)
- net BTN_PWR: now also IC3.12 (PA0)
- net BTN_RIGHT: now also IC3.11 (PC3)
- net BTN_UP: now also IC3.8 (PC0)
- net GND: now also IC3.15 (VSS_1), IC3.27 (VSSA), IC3.31 (VSS_2), IC3.47 (VSS_3), IC3.63 (VSS_4)
- net OLED_CLK: now also IC3.19 (PA5)
- net OLED_CS: now also IC3.18 (PA4)
- net OLED_DC: now also IC3.30 (PB10)
- net OLED_DIN: now also IC3.21 (PA7)
- net OLED_RST: now also IC3.22 (PC4)
- net nRESET: now also IC3.7 (PG10-NRST)
- net at C16.1, Y1.3: now also IC3.5 (PF0-OSC_IN)
- net at C17.2, Y1.1: now also IC3.6 (PF1-OSC_OUT)

Commit message: Added power enable logic
Parts:
- added R?: 10K, Resistor_SMD:R_0402_1005Metric_Pad0.72x0.64mm_HandSolder, symbol Device:R_Small
- C16: value 10nF -> (none); footprint Capacitor_SMD:C_0402_1005Metric_Pad0.74x0.62mm_HandSolder -> (none)
Connections:
- net +3V3: now also R?.1
- net JTAG_TCK: now also IC3.50 (PA14)
- net JTAG_TDI: now also IC3.51 (PA15)
- net JTAG_TDO: now also IC3.56 (PB3)
- net JTAG_TMS: now also IC3.49 (PA13)
- net PSU_EN: now reaches IC3.46 (PA12)
- net PSU_EN: now also R?.2
Changed lines of the file:
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@@
   (junction (at 88.265 177.8) (diameter 0) (color 0 0 0 0)
   )
+  (junction (at 198.755 85.09) (diameter 0) (color 0 0 0 0)
+  )
   (junction (at 109.855 177.8) (diameter 0) (color 0 0 0 0)
   )
@@
     (stroke (width 0) (type default) (color 0 0 0 0))
   )
+  (wire (pts (xy 198.755 82.55) (xy 198.755 85.09))
+    (stroke (width 0) (type default) (color 0 0 0 0))
+  )
   (wire (pts (xy 99.06 177.8) (xy 109.855 177.8))
     (stroke (width 0) (type default) (color 0 0 0 0))
@@
     (stroke (width 0) (type default) (color 0 0 0 0))
   )
+  (wire (pts (xy 198.755 85.09) (xy 182.88 85.09))
+    (stroke (width 0) (type default) (color 0 0 0 0))
+  )
   (wire (pts (xy 32.385 38.1) (xy 42.545 38.1))
     (stroke (width 0) (type default) (color 0 0 0 0))
@@
     (stroke (width 0) (type default) (color 0 0 0 0))
   )
+  (wire (pts (xy 208.915 85.09) (xy 198.755 85.09))
+    (stroke (width 0) (type default) (color 0 0 0 0))
+  )
   (bus (pts (xy 29.845 30.48) (xy 29.845 33.02))
     (stroke (width 0) (type default) (color 0 0 0 0))
@@
     (effects (font (size 1.27 1.27)) (justify left bottom))
   )
-  (label "JTAG_TDI" (at 151.765 59.69 90)
+  (label "JTAG_TDI" (at 165.1 66.04 90)
     (effects (font (size 1.27 1.27)) (justify left bottom))
   )
@@
     (effects (font (size 1.27 1.27)) (justify left bottom))
   )
-  (label "JTAG_TDO" (at 154.305 59.69 90)
+  (label "JTAG_TDO" (at 152.4 66.04 90)
     (effects (font (size 1.27 1.27)) (justify left bottom))
   )
@@
     (effects (font (size 1.27 1.27)) (justify left bottom))
   )
-  (label "JTAG_TCK" (at 156.845 59.69 90)
-    (effects (font (size 1.27 1.27)) (justify left bottom))
-  )
-  (label "JTAG_TMS" (at 159.385 59.69 90)
+  (label "JTAG_TCK" (at 167.64 66.04 90)
+    (effects (font (size 1.27 1.27)) (justify left bottom))
+  )
+  (label "JTAG_TMS" (at 170.18 66.04 90)
     (effects (font (size 1.27 1.27)) (justify left bottom))
   )
@@
     (effects (font (size 1.27 1.27)) (justify right))
   )
+  (hierarchical_label "PSU_EN" (shape output) (at 208.915 85.09 0)
+    (effects (font (size 1.27 1.27)) (justify left))
+  )
   (hierarchical_label "{USB" (shape input) (at 20.955 99.06 180)
     (effects (font (size 1.27 1.27)) (justify right))
@@
     )
     (property "Datasheet" "" (id 3) (at 85.09 91.44 0)
+      (effects (font (size 1.27 1.27)) hide)
+    )
+    (pin "1")
+  )
+  (symbol (lib_id "power:+3.3V") (at 198.755 77.47 0) (unit 1)
+    (in_bom yes) (on_board yes)
+    (property "Reference" "#PWR?" (id 0) (at 198.755 81.28 0)
+      (effects (font (size 1.27 1.27)) hide)
+    )
+    (property "Value" "+3.3V" (id 1) (at 198.755 68.58 90)
+      (effects (font (size 1.27 1.27)) (justify right))
+    )
+    (property "Footprint" "" (id 2) (at 198.755 77.47 0)
+      (effects (font (size 1.27 1.27)) hide)
+    )
+    (property "Datasheet" "" (id 3) (at 198.755 77.47 0)
       (effects (font (size 1.27 1.27)) hide)
     )
@@
     (pin "2")
   )
+  (symbol (lib_id "Device:R_Small") (at 198.755 80.01 0) (unit 1)
+    (in_bom yes) (on_board yes) (fields_autoplaced)
+    (property "Reference" "R?" (id 0) (at 200.2536 79.1753 0)
+      (effects (font (size 1.27 1.27)) (justify left))
+    )
+    (property "Value" "10K" (id 1) (at 200.2536 81.7122 0)
+      (effects (font (size 1.27 1.27)) (justify left))
+    )
+    (property "Footprint" "Resistor_SMD:R_0402_1005Metric_Pad0.72x0.64mm_HandSolder" (id 2) (at 198.755 80.01 0)
+      (effects (font (size 1.27 1.27)) hide)
+    )
+    (property "Datasheet" "~" (id 3) (at 198.755 80.01 0)
+      (effects (font (size 1.27 1.27)) hide)
+    )
+    (pin "1")
+    (pin "2")
+  )
   (symbol (lib_id "Device:C_Small") (at 90.17 97.79 180) (unit 1)
     (in_bom yes) (on_board yes) (fields_autoplaced)
@@
       (effects (font (size 1.27 1.27)) (justify right))
     )
-    (property "Value" "10nF" (id 1) (at 92.4941 86.7858 0)
-      (effects (font (size 1.27 1.27)) (justify right))
-    )
-    (property "Footprint" "Capacitor_SMD:C_0402_1005Metric_Pad0.74x0.62mm_HandSolder" (id 2) (at 90.17 85.09 0)
-      (effects (font (size 1.27 1.27)) hide)
-    )
+    (property "Value" "" (id 1) (at 92.4941 86.7858 0)
+      (effects (font (size 1.27 1.27)) (justify right))
+    )
+    (property "Footprint" "" (id 2) (at 90.17 85.09 0)
+      (effects (font (size 1.27 1.27)) hide)
+    )
